File: AMShieldV1/ChickenDoor_V1.kicad_pcb (KiCad board)
At the start: 2 copper layers, 100 x 100 mm, 37 parts, among them J1 Screw_Terminal_01x03, J2 Screw_Terminal_01x02, J3 Screw_Terminal_01x02, J4 Screw_Terminal_01x02, J7 Screw_Terminal_01x02, K1 FINDER-36.11, K2 FINDER-36.11, K3 FINDER-36.11, Q1 BC547, Q2 BC547, Q3 BC547, Q4 BC557, SW1 SW_Push, SW2 SW_Push, SW3 SW_Push, SW4 SW_Push

Commit message: First draft of the PCB with updated schematic.
Parts:
- removed REF**: CR2013-MI2120, Display:CR2013-MI2120
- removed XA1: Arduino_Mega2560_Shield, arduino:Arduino_Mega2560_Shield
- added H1: MountingHole, MountingHole:MountingHole_4.3mm_M4_DIN965, F.Cu at (55.0, 65.0)
- added H2: MountingHole, MountingHole:MountingHole_4.3mm_M4_DIN965, F.Cu at (135.0, 65.0)
- added H3: MountingHole, MountingHole:MountingHole_4.3mm_M4_DIN965, F.Cu at (135.0, 145.0)
- added H4: MountingHole, MountingHole:MountingHole_4.3mm_M4_DIN965, F.Cu at (56.0, 145.0)
- added J6: KMR-1.8 SPI, KMR-1:KMR-1.8-SPI, F.Cu at (76.5, 111.0)
- added JP1: SolderJumper_2_Bridged, Jumper:SolderJumper-2_P1.3mm_Bridged_RoundedPad1.0x1.5mm, F.Cu at (95.3, 87.6)
- added JP2: SolderJumper_2_Bridged, Jumper:SolderJumper-2_P1.3mm_Bridged_RoundedPad1.0x1.5mm, F.Cu at (95.3, 90.8)
- added JP3: SolderJumper_2_Bridged, Jumper:SolderJumper-2_P1.3mm_Bridged_RoundedPad1.0x1.5mm, F.Cu at (95.2, 94.0)
- added JP4: SolderJumper_2_Bridged, Jumper:SolderJumper-2_P1.3mm_Bridged_RoundedPad1.0x1.5mm, F.Cu at (95.2, 97.2)
- added U1: MEGA_PRO_EMBED_CH340G___ATMEGA2560, MEGA_PRO_EMBED_CH340G___ATMEGA2560:MODULE_MEGA_PRO_EMBED_CH340G___ATMEGA2560, B.Cu at (112.6, 92.1)
- added U2: TC00500, TC00500_DS3231_AT24C32:MODULE_TC00500_FHk_BatteryUpside, F.Cu at (62.9, 73.7)
- D1, D3: footprint LED_THT:LED_D5.0mm -> LED_SMD:LED_1206_3216Metric
- D2, D6: value 1N4148 -> 1N4448W; footprint Diode_THT:D_DO-35_SOD27_P7.62mm_Horizontal -> Diode_SMD:D_SOD-123
- D4: value 1N4148 -> LED; footprint Diode_THT:D_DO-35_SOD27_P7.62mm_Horizontal -> LED_SMD:LED_1206_3216Metric
- D5: value LED -> 1N4448W; footprint LED_THT:LED_D5.0mm -> Diode_SMD:D_SOD-123
- J1: footprint TerminalBlock_MetzConnect:TerminalBlock_MetzConnect_Type011_RT05503HBWC_1x03_P5.00mm_Horizontal -> TerminalBlock_Phoenix:TerminalBlock_Phoenix_MKDS-1,5-3-5.08_1x03_P5.08mm_Horizontal
- J2, J3, J4, J7: footprint TerminalBlock_MetzConnect:TerminalBlock_MetzConnect_Type011_RT05502HBWC_1x02_P5.00mm_Horizontal -> TerminalBlock_Phoenix:TerminalBlock_Phoenix_MKDS-1,5-2-5.08_1x02_P5.08mm_Horizontal
- Q1, Q2, Q3: value BC547 -> BC817; footprint Package_TO_SOT_THT:TO-92_Inline -> Package_TO_SOT_SMD:SOT-23
- Q4: value BC557 -> BC807; footprint Package_TO_SOT_THT:TO-92_Inline -> Package_TO_SOT_SMD:SOT-23
- R1, R2, R3, R4: footprint Resistor_THT:R_Axial_DIN0207_L6.3mm_D2.5mm_P10.16mm_Horizontal -> Resistor_SMD:R_0805_2012Metric
- R5, R6: value 2k2 -> 560; footprint Resistor_THT:R_Axial_DIN0207_L6.3mm_D2.5mm_P10.16mm_Horizontal -> Resistor_SMD:R_0805_2012Metric
- R7: value 560 -> 2k2; footprint Resistor_THT:R_Axial_DIN0207_L6.3mm_D2.5mm_P10.16mm_Horizontal -> Resistor_SMD:R_0805_2012Metric
- R8: value 560 -> 18R; footprint Resistor_THT:R_Axial_DIN0207_L6.3mm_D2.5mm_P10.16mm_Horizontal -> Resistor_SMD:R_0805_2012Metric
- R9: value 18R -> 2k2; footprint Resistor_THT:R_Axial_DIN0207_L6.3mm_D2.5mm_P10.16mm_Horizontal -> Resistor_SMD:R_0805_2012Metric
- moved K3 225.9 mm to (119.2, 133.7)
- moved D6 218.1 mm to (114.5, 128.6)
- moved Q3 208.6 mm to (102.7, 128.6), turned to 270 degrees
- moved D5 207.6 mm to (92.3, 128.6), turned to 0 degrees
- moved J3 200.8 mm to (58.1, 161.4)
- moved J1 198.7 mm to (85.6, 161.4)
- moved D8 198.0 mm to (120.0, 163.6), turned to 270 degrees
- moved D10 191.3 mm to (115.6, 163.6), turned to 270 degrees
- moved R1 191.2 mm to (75.4, 128.6)
- moved J4 191.1 mm to (70.5, 161.4)
- moved R3 190.3 mm to (97.6, 128.6), turned to 180 degrees
- moved Q2 189.0 mm to (124.9, 128.6), turned to 270 degrees
- moved R4 187.6 mm to (119.8, 128.6), turned to 180 degrees
- moved D7 187.4 mm to (120.0, 156.6), turned to 270 degrees
- moved J7 187.0 mm to (127.5, 161.5)
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Connections:
- D4 pad 1: +5V -> Net-(D4-Pad1)
- D4 pad 2: Net-(D4-Pad2) -> +5V
- D5 pad 1: Net-(D5-Pad1) -> +5V
- D5 pad 2: +5V -> Net-(D5-Pad2)
- K1 pad 11: Net-(D7-Pad2) -> Net-(J1-Pad2)
- K1 pad 12: Net-(D10-Pad2) -> Net-(J1-Pad3)
- K1 pad 14: Net-(D7-Pad1) -> Net-(J1-Pad1)
- K2 pad 11: Net-(D10-Pad1) -> Net-(D7-Pad2)
- K2 pad A2: Net-(D4-Pad2) -> Net-(D5-Pad2)
- K3 pad 11: Net-(J1-Pad2) -> Net-(D10-Pad1)
- K3 pad 12: Net-(J1-Pad3) -> Net-(D10-Pad2)
- K3 pad 14: Net-(J1-Pad1) -> Net-(D7-Pad1)
- Q1 pad 1: Net-(D2-Pad2) -> Net-(Q1-Pad1)
- Q1 pad 2: Net-(Q1-Pad2) -> GND
- Q1 pad 3: GND -> Net-(D2-Pad2)
- Q2 pad 1: Net-(D4-Pad2) -> Net-(Q2-Pad1)
- Q2 pad 2: Net-(Q2-Pad2) -> GND
- Q2 pad 3: GND -> Net-(D6-Pad2)
- Q3 pad 1: Net-(D6-Pad2) -> Net-(Q3-Pad1)
- Q3 pad 2: Net-(Q3-Pad2) -> GND
- Q3 pad 3: GND -> Net-(D5-Pad2)
- Q4 pad 2: Net-(Q4-Pad2) -> +5V
- Q4 pad 3: +5V -> Net-(Q4-Pad3)
- R1 pad 1: Net-(Q3-Pad2) -> Net-(Q1-Pad1)
- R2 pad 1: Net-(D6-Pad2) -> Net-(D2-Pad2)
- R2 pad 2: Net-(D5-Pad1) -> Net-(D1-Pad1)
- R3 pad 1: Net-(Q1-Pad2) -> Net-(Q3-Pad1)
- R4 pad 1: Net-(Q2-Pad2) -> Net-(Q2-Pad1)
- R5 pad 1: +5V -> Net-(D5-Pad2)
- R5 pad 2: /TFT_reset -> Net-(D3-Pad1)
- R6 pad 1: Net-(Q4-Pad2) -> Net-(D6-Pad2)
- R6 pad 2: /TFT_Dimming -> Net-(D4-Pad1)
- R7 pad 1: Net-(D2-Pad2) -> Net-(Q4-Pad1)
- R7 pad 2: Net-(D1-Pad1) -> /TFT_Dimming
- R8 pad 1: Net-(D4-Pad2) -> Net-(J6-Pad15)
- R8 pad 2: Net-(D3-Pad1) -> Net-(Q4-Pad3)
- R9 pad 1: Net-(J6-Pad15) -> +5V
- R9 pad 2: Net-(Q4-Pad1) -> /TFT_reset
Routing:
- net +5V: track 0.00 -> 266.3 mm, vias 0 -> 7
- net /RTC_SCL: track 0.00 -> 90.1 mm
- net /RTC_SDA: track 0.00 -> 85.6 mm
- net /DoorPositionDown: track 0.00 -> 78.3 mm
- net /DoorPositionUp: track 0.00 -> 78.2 mm
- net GND: track 0.00 -> 76.6 mm, vias 0 -> 6
- net /IndoorLighting: track 0.00 -> 60.6 mm, vias 0 -> 2
- net /TFT_CS: track 0.00 -> 52.1 mm, vias 0 -> 1
- net Net-(D10-Pad2): track 0.00 -> 52.0 mm, vias 0 -> 1
- net /TFT_DataOrCommand: track 0.00 -> 51.1 mm, vias 0 -> 1
- net Net-(D7-Pad2): track 0.00 -> 50.5 mm, vias 0 -> 1
- net /TFT_reset: track 0.00 -> 50.3 mm, vias 0 -> 2
- net Net-(D7-Pad1): track 0.00 -> 49.8 mm, vias 0 -> 2
- net Net-(D10-Pad1): track 0.00 -> 49.6 mm, vias 0 -> 1
- net /TFT_Dimming: track 0.00 -> 39.6 mm, vias 0 -> 1
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- added copper zone on B.Cu, net GND
Other:
- board size 100 x 100 mm -> 90 x 110 mm
- net class Power added: clearance 0.2, trace_width 1.5, via_dia 0.8, via_drill 0.4
- board text added: "(Lamp)"
- board text added: "(Motor)"
- board text added: "+ -"
- board text added: "Down"
- board text added: "Down pos"
- board text added: "Funky Chicken Door v. 1.0.0"
- board text added: "Light"
- board text added: "Motor"
- board text added: "NO COM NC"
- board text added: "RTC-DS3231"
- board text added: "Up"
- board text added: "Up pos"
